File: KiCad/PowerDistrubutionBoard/PowerDistrubutionBoard.kicad_pcb (KiCad board)
At the start: 2 copper layers, 77 x 18.5 mm, 10 parts, among them J1 BEC, J2 RS_OUT, J4 R-, J5 R+, J6 RS, T1 PWR_D1, T2 PWR_D2, T3 PWR_IN, T4 PWR_W

Commit message: new stuff
Parts:
- removed J2: RS_OUT, Connector_PinHeader_2.54mm:PinHeader_1x06_P2.54mm_Vertical
- removed J4: R-, Connector_PinHeader_2.54mm:PinHeader_1x07_P2.54mm_Vertical
- added J10: Batt, Connector_PinHeader_2.54mm:PinHeader_1x03_P2.54mm_Vertical, F.Cu at (103.8, 54.7)
- added J7: S_Out, Connector_PinHeader_2.54mm:PinHeader_2x04_P2.54mm_Horizontal, F.Cu at (154.2, 53.8)
- added J8: Ch3, Connector_PinHeader_2.54mm:PinHeader_1x03_P2.54mm_Vertical, F.Cu at (94.5, 54.7)
- added J9: Ch4, Connector_PinHeader_2.54mm:PinHeader_1x03_P2.54mm_Vertical, F.Cu at (99.2, 54.7)
- J1: footprint Connector_PinHeader_2.00mm:PinHeader_1x04_P2.00mm_Vertical -> Connector_PinHeader_2.54mm:PinHeader_1x04_P2.54mm_Vertical
- J5: value R+ -> Ch1; footprint Connector_PinHeader_2.54mm:PinHeader_1x07_P2.54mm_Vertical -> Connector_PinHeader_2.54mm:PinHeader_1x03_P2.54mm_Vertical
- J6: value RS -> Ch2; footprint Connector_PinHeader_2.54mm:PinHeader_1x07_P2.54mm_Vertical -> Connector_PinHeader_2.54mm:PinHeader_1x03_P2.54mm_Vertical
- moved T1 50.9 mm to (161.8, 59.4), turned to -90 degrees
- moved S1 46.1 mm to (198.8, 62.4)
- moved T4 41.6 mm to (180.9, 60.4)
- moved T2 38.0 mm to (155.4, 59.4), turned to -90 degrees
- moved J5 37.1 mm to (85.2, 54.7)
- moved T3 36.4 mm to (197.2, 60.6), turned to 0 degrees
- moved J6 34.0 mm to (89.8, 54.7)
- moved J1 25.7 mm to (128.0, 62.1), turned to 180 degrees
Connections:
- J1 pad 1: Net-(J1-Pad1) -> Net-(J1-Pin_1)
- J1 pad 2: Net-(J1-Pad2) -> Net-(J1-Pin_2)
- J1 pad 3: Net-(J1-Pad3) -> Net-(J1-Pin_3)
- J1 pad 4: Net-(J1-Pad4) -> unconnected-(J1-Pin_4-Pad4)
- J5 pad 1: Net-(J1-Pad4) -> Net-(J1-Pin_3)
- J5 pad 3: unconnected-(J5-Pad3) -> Net-(J5-Pin_3)
- J6 pad 1: unconnected-(J6-Pad1) -> Net-(J1-Pin_3)
- J6 pad 2: Net-(J2-Pad1) -> unconnected-(J6-Pin_2-Pad2)
- S1 pad 1: Net-(T3-Pad1) -> Net-(T3--)
- S1 pad 2: Net-(J1-Pad1) -> Net-(J1-Pin_2)
- T1 pad 1: Net-(J1-Pad1) -> Net-(J1-Pin_1)
- T1 pad 2: Net-(J1-Pad2) -> Net-(J1-Pin_2)
- T2 pad 1: Net-(J1-Pad1) -> Net-(J1-Pin_1)
- T2 pad 2: Net-(J1-Pad2) -> Net-(J1-Pin_2)
- T3 pad 1: Net-(T3-Pad1) -> Net-(J1-Pin_1)
- T3 pad 2: Net-(J1-Pad2) -> Net-(T3--)
- T4 pad 1: Net-(J1-Pad1) -> Net-(J1-Pin_1)
- T4 pad 2: Net-(J1-Pad2) -> Net-(J1-Pin_2)
Routing:
- net Net-(J2-Pad1): track 39.4 -> 0.00 mm
- net Net-(J6-Pin_3): track 37.8 -> 0.00 mm
- net Net-(J2-Pad3): track 36.4 -> 0.00 mm
- net Net-(J2-Pad4): track 34.9 -> 0.00 mm
- net Net-(J2-Pad5): track 33.3 -> 0.00 mm
- net Net-(J2-Pad6): track 31.5 -> 0.00 mm
- net Net-(J1-Pad4): track 25.4 -> 0.00 mm
- net Net-(J1-Pad3): track 23.0 -> 0.00 mm
- net Net-(J1-Pad2): track 22.2 -> 0.00 mm
- net Net-(J1-Pad1): track 11.2 -> 0.00 mm
- removed copper zone on B.Cu, net Net-(J1-Pad1)
- removed copper zone on F.Cu, net Net-(J1-Pad2)
- removed copper zone on F.Cu, net Net-(T3-Pad1)
Other:
- board size 77 x 18.5 mm -> 90 x 15 mm

Commit message: adds maore stuff
Parts:
- moved J5 37.6 mm to (122.7, 56.7), turned to -90 degrees
- moved J6 33.2 mm to (122.7, 59.5), turned to -90 degrees
- moved J8 29.2 mm to (122.7, 62.3), turned to -90 degrees
- moved T2 27.7 mm to (181.8, 67.7), turned to 0 degrees
- moved J7 26.3 mm to (128.1, 57.2), turned to 0 degrees
- moved J1 26.3 mm to (152.2, 51.9), turned to -90 degrees
- moved J9 25.7 mm to (122.7, 65.1), turned to -90 degrees
- moved T1 20.1 mm to (181.8, 60.7), turned to 0 degrees
- moved T4 19.4 mm to (161.6, 60.6)
- moved J10 18.9 mm to (122.7, 53.9), turned to -90 degrees
- moved S1 0.84 mm to (199.5, 62.8)
Connections:
- J1 pad 4: unconnected-(J1-Pin_4-Pad4) -> Net-(J1-Pin_4)
- J10 pad 2: unconnected-(J10-Pin_2-Pad2) -> Net-(J1-Pin_4)
- J5 pad 2: unconnected-(J5-Pin_2-Pad2) -> Net-(J1-Pin_4)
- J6 pad 2: unconnected-(J6-Pin_2-Pad2) -> Net-(J1-Pin_4)
- J8 pad 2: unconnected-(J8-Pin_2-Pad2) -> Net-(J1-Pin_4)
- J9 pad 2: unconnected-(J9-Pin_2-Pad2) -> Net-(J1-Pin_4)
- S1 pad 1: Net-(T3--) -> Net-(J1-Pin_2)
Routing:
- net Net-(J1-Pin_4): track 0.00 -> 36.3 mm
- net Net-(J6-Pin_3): track 0.00 -> 11.7 mm
- net Net-(J7-Pin_7): track 0.00 -> 11.6 mm
- net Net-(J7-Pin_5): track 0.00 -> 11.5 mm
- net Net-(J5-Pin_3): track 0.00 -> 11.2 mm
- net Net-(T3--): track 0.00 -> 7.27 mm
- added copper zone on B.Cu, net Net-(J1-Pin_1)
- added copper zone on F.Cu, net Net-(J1-Pin_2)
- added copper zone on B.Cu, net Net-(J1-Pin_3)
