File: KiCad/PowerDistrubutionBoard/PowerDistrubutionBoard.kicad_sch (KiCad schematic)
At the start: 10 parts, among them J1 BEC, J2 RS_OUT, J4 R-, J5 R+, J6 RS, T1 PWR_D1, T2 PWR_D2, T3 PWR_IN, T4 PWR_W

Commit message: new stuff
Parts:
- removed J1: BEC, Connector_PinHeader_2.00mm:PinHeader_1x04_P2.00mm_Vertical, symbol Connector:Conn_01x04_Female
- removed J2: RS_OUT, Connector_PinHeader_2.54mm:PinHeader_1x06_P2.54mm_Vertical, symbol Connector:Conn_01x06_Male
- removed J4: R-, Connector_PinHeader_2.54mm:PinHeader_1x07_P2.54mm_Vertical, symbol Connector:Conn_01x07_Female
- removed J5: R+, Connector_PinHeader_2.54mm:PinHeader_1x07_P2.54mm_Vertical, symbol Connector:Conn_01x07_Female
- removed J6: RS, Connector_PinHeader_2.54mm:PinHeader_1x07_P2.54mm_Vertical, symbol Connector:Conn_01x07_Female
- added J1: BEC, Connector_PinHeader_2.54mm:PinHeader_1x04_P2.54mm_Vertical, symbol Connector:Conn_01x04_Socket
- added J10: Batt, Connector_PinHeader_2.54mm:PinHeader_1x03_P2.54mm_Vertical, symbol Connector_Generic:Conn_01x03
- added J5: Ch1, Connector_PinHeader_2.54mm:PinHeader_1x03_P2.54mm_Vertical, symbol Connector_Generic:Conn_01x03
- added J6: Ch2, Connector_PinHeader_2.54mm:PinHeader_1x03_P2.54mm_Vertical, symbol Connector_Generic:Conn_01x03
- added J7: S_Out, Connector_PinHeader_2.54mm:PinHeader_2x04_P2.54mm_Horizontal, symbol Connector_Generic:Conn_02x04_Odd_Even
- added J8: Ch3, Connector_PinHeader_2.54mm:PinHeader_1x03_P2.54mm_Vertical, symbol Connector_Generic:Conn_01x03
- added J9: Ch4, Connector_PinHeader_2.54mm:PinHeader_1x03_P2.54mm_Vertical, symbol Connector_Generic:Conn_01x03
Connections:
- net at T1.1 (+), T2.1 (+), T4.1 (+): now also T3.1 (+), J1.1 (Pin_1); no longer S1.2
- net at T1.2 (-), T2.2 (-), T4.2 (-): now also S1.2, J1.2 (Pin_2); no longer T3.2 (-)
- net at S1.1: now also T3.2 (-); no longer T3.1 (+)
- new net: J1.3 (Pin_3), J10.1 (Pin_1), J5.1 (Pin_1), J6.1 (Pin_1), J7.2 (Pin_2), J7.4 (Pin_4), J7.6 (Pin_6), J7.8 (Pin_8), J8.1 (Pin_1), J9.1 (Pin_1)
- new net: J7.5 (Pin_5), J8.3 (Pin_3)
- new net: J7.7 (Pin_7), J9.3 (Pin_3)
- new net: J5.3 (Pin_3), J7.1 (Pin_1)
- new net: J6.3 (Pin_3), J7.3 (Pin_3)
- no-connect marks 13 -> 0
Other:
- moved on the sheet: S1, T1, T2, T3, T4

Commit message: adds maore stuff
Connections:
- net at J8.2 (Pin_2): now also J1.4 (Pin_4), J10.2 (Pin_2), J5.2 (Pin_2), J6.2 (Pin_2), J9.2 (Pin_2)
Changed lines of the file:
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@@
 (kicad_sch (version 20230121) (generator eeschema)
   (paper "A4")
+  (junction (at 78.74 88.9) (diameter 0) (color 0 0 0 0)
+  )
   (junction (at 147.32 87.63) (diameter 0) (color 0 0 0 0)
+  )
+  (junction (at 106.68 88.9) (diameter 0) (color 0 0 0 0)
+  )
+  (junction (at 64.77 88.9) (diameter 0) (color 0 0 0 0)
   )
   (junction (at 34.29 76.2) (diameter 0) (color 0 0 0 0)
@@
   )
   (junction (at 34.29 78.74) (diameter 0) (color 0 0 0 0)
+  )
+  (junction (at 92.71 88.9) (diameter 0) (color 0 0 0 0)
   )
   (junction (at 165.1 74.93) (diameter 0) (color 0 0 0 0)
@@
     (stroke (width 0) (type default))
   )
+  (wire (pts (xy 92.71 88.9) (xy 106.68 88.9))
+    (stroke (width 0) (type default))
+  )
   (wire (pts (xy 34.29 81.28) (xy 34.29 87.63))
     (stroke (width 0) (type default))
@@
     (stroke (width 0) (type default))
   )
+  (wire (pts (xy 92.71 91.44) (xy 92.71 88.9))
+    (stroke (width 0) (type default))
+  )
   (wire (pts (xy 127 87.63) (xy 133.35 87.63))
     (stroke (width 0) (type default))
@@
   )
   (wire (pts (xy 124.46 91.44) (xy 124.46 74.93))
+    (stroke (width 0) (type default))
+  )
+  (wire (pts (xy 78.74 91.44) (xy 78.74 88.9))
     (stroke (width 0) (type default))
   )
@@
     (stroke (width 0) (type default))
   )
+  (wire (pts (xy 64.77 91.44) (xy 64.77 88.9))
+    (stroke (width 0) (type default))
+  )
   (wire (pts (xy 76.2 91.44) (xy 76.2 78.74))
     (stroke (width 0) (type default))
@@
     (stroke (width 0) (type default))
   )
+  (wire (pts (xy 50.8 88.9) (xy 64.77 88.9))
+    (stroke (width 0) (type default))
+  )
   (wire (pts (xy 121.92 91.44) (xy 121.92 87.63))
+    (stroke (width 0) (type default))
+  )
+  (wire (pts (xy 78.74 88.9) (xy 92.71 88.9))
     (stroke (width 0) (type default))
   )
@@
   )
   (wire (pts (xy 95.25 87.63) (xy 109.22 87.63))
+    (stroke (width 0) (type default))
+  )
+  (wire (pts (xy 50.8 91.44) (xy 50.8 88.9))
     (stroke (width 0) (type default))
   )
@@
   )
   (wire (pts (xy 34.29 73.66) (xy 34.29 76.2))
+    (stroke (width 0) (type default))
+  )
+  (wire (pts (xy 119.38 88.9) (xy 106.68 88.9))
+    (stroke (width 0) (type default))
+  )
+  (wire (pts (xy 106.68 88.9) (xy 106.68 91.44))
     (stroke (width 0) (type default))
   )
@@
     (stroke (width 0) (type default))
   )
+  (wire (pts (xy 64.77 88.9) (xy 78.74 88.9))
+    (stroke (width 0) (type default))
+  )
